File: hardware/balloon_board/BalloonBoard.sch (EAGLE design)
At the start: 35 parts, among them IC1 TLC274P, J1 Com 4, J2 Com 3, J3 22-27-2021-02

Commit message: new layout with gyro and pressure sensor
Parts:
- removed C4: 470p, resistor:C-EU025-024X044
- removed C5: 10n, capacitor-wima:C2.5/2
- removed PS1: MPX5100DP, mpx-freescale:MPX5010DP-V
- removed R19: 22k, resistor:R-EU_0207/10
- removed R20: 68k, resistor:R-EU_0207/10
- added U$1: PRESSUREMODULE, SpaceBallonV3:PRESSUREMODULE
- added U$2: MPU-6050, SpaceBallonV3:MPU-6050
- R15: device resistor:R-EU_0207/10 -> resistor:R-EU_0207/12
Connections:
- new net +3V3_B: JP4.5, U$2.VDD, U$2.VLOGIC
- new net N$26: JP6.22, U$1.RX
- new net N$27: JP6.24, U$1.TX
- net +3V3: now also JP6.1, U$1.+3.3V; no longer JP4.5
- net +5V: now also JP6.39; no longer C5.1, JP4.4, PS1.VS
- net GND: now also JP6.38, U$1.GND, U$1.SPISEL, U$2.GND; no longer C4.2, C5.2, PS1.GND, R20.1
- net N$17: now also JP5.8; no longer JP5.7
- net N$18: now also JP5.7; no longer JP5.8
- net N$20: now also JP5.6, U$2.SDA; no longer JP3.3, R19.1, R20.2
- net N$25: now also JP5.5, U$2.SCL; no longer C4.1, PS1.VOUT, R19.2
Other:
- note added: "Com 2"
- moved on the sheet: C1, J1-1, J1-2, J1-3, J1-4, J2-1, J2-2, J2-3, J2-4, JP5, JP6
